File: pcb/v1/v1.kicad_sch (KiCad schematic)
At the start: 0 parts

Commit message: First pcb schematic
Parts:
- added C1, C2: 10u, symbol Device:C_Small
- added C10, C13, C14, C3, C4, C5, C6, C7, C8, C9: 100n, symbol Device:C_Small
- added C11, C12: 1u, symbol Device:C_Small
- added D1, D10, D11, D12, D13, D14, D15, D16, D17, D18, D19, D2, D20, D21, D22, D23, D24, D25, D26, D27, D28, D29, D3, D30, D31, D32, D33, D34, D35, D36, D37, D38, D39, D4, D40, D41, D42, D44, D45, D46, D47, D48, D5, D6, D7, D8, D9: D_Small, symbol Device:D_Small
- added J1: USB_C_Receptacle_USB2.0_16P, symbol Connector:USB_C_Receptacle_USB2.0_16P
- added R1, R2: 5k1, symbol Device:R_Small
- added R3, R4: 27.4, symbol Device:R_Small
- added SW1, SW10, SW11, SW12, SW13, SW14, SW15, SW16, SW17, SW18, SW19, SW2, SW20, SW21, SW22, SW23, SW24, SW25, SW26, SW27, SW28, SW29, SW3, SW30, SW31, SW32, SW33, SW34, SW35, SW36, SW37, SW38, SW39, SW4, SW40, SW41, SW42, SW44, SW45, SW46, SW47, SW48, SW5, SW6, SW7, SW8, SW9: SW_SPST, symbol Switch:SW_SPST
- added U1: RP2040, Package_DFN_QFN:QFN-56-1EP_7x7mm_P0.4mm_EP3.2x3.2mm, symbol MCU_RaspberryPi:RP2040
- added U2: USB6B1, Package_SO:SOIC-8_3.9x4.9mm_P1.27mm, symbol Power_Protection:USB6B1
- added U3: NCP1117-3.3_SOT223, Package_TO_SOT_SMD:SOT-223-3_TabPin2, symbol Regulator_Linear:NCP1117-3.3_SOT223
Connections:
- new net: J1.A7 (D-), J1.B7 (D-), U2.2 (I/O1)
- new net: J1.A6 (D+), J1.B6 (D+), U2.3 (I/O2)
- new net: D11.2 (A), SW11.1 (A)
- new net: D15.2 (A), SW15.1 (A)
- new net: D22.2 (A), SW22.1 (A)
- new net: D30.2 (A), SW30.1 (A)
- new net: D46.2 (A), SW46.1 (A)
- new net: D37.2 (A), SW37.1 (A)
- new net: D12.2 (A), SW12.1 (A)
- new net: D9.2 (A), SW9.1 (A)
- new net: D47.2 (A), SW47.1 (A)
- new net: D44.2 (A), SW44.1 (A)
- new net: D2.2 (A), SW2.1 (A)
- new net: D3.2 (A), SW3.1 (A)
- new net: D14.2 (A), SW14.1 (A)
- new net: D38.2 (A), SW38.1 (A)
- new net: D27.2 (A), SW27.1 (A)
- new net: D8.2 (A), SW8.1 (A)
- new net: D4.2 (A), SW4.1 (A)
- new net: D31.2 (A), SW31.1 (A)
- new net: J1.A5 (CC1), R1.1
- new net: J1.B5 (CC2), R2.1
- new net: D25.2 (A), SW25.1 (A)
- new net: R4.2, U1.47 (USB_DP)
- new net: D36.2 (A), SW36.1 (A)
- new net: D48.2 (A), SW48.1 (A)
- new net: D6.2 (A), SW6.1 (A)
- new net: D42.2 (A), SW42.1 (A)
- new net: D29.2 (A), SW29.1 (A)
- new net: D34.2 (A), SW34.1 (A)
- new net: D35.2 (A), SW35.1 (A)
- new net: R3.2, U1.46 (USB_DM)
- new net: D20.2 (A), SW20.1 (A)
- new net: D10.2 (A), SW10.1 (A)
- new net: D13.2 (A), SW13.1 (A)
- new net: D28.2 (A), SW28.1 (A)
- new net: D16.2 (A), SW16.1 (A)
- new net: D26.2 (A), SW26.1 (A)
- new net: D17.2 (A), SW17.1 (A)
- new net: D41.2 (A), SW41.1 (A)
- new net: D24.2 (A), SW24.1 (A)
- new net: D18.2 (A), SW18.1 (A)
- new net: D39.2 (A), SW39.1 (A)
- new net: D7.2 (A), SW7.1 (A)
- new net: D33.2 (A), SW33.1 (A)
- new net: D23.2 (A), SW23.1 (A)
- new net: D40.2 (A), SW40.1 (A)
- new net: D5.2 (A), SW5.1 (A)
- new net: D32.2 (A), SW32.1 (A)
- new net: D21.2 (A), SW21.1 (A)
- new net: D45.2 (A), SW45.1 (A)
- new net: D1.2 (A), SW1.1 (A)
- new net: D19.2 (A), SW19.1 (A)
- new net +1V1: C12.1, C13.1, C14.1, U1.23 (DVDD), U1.45 (VREG_VOUT), U1.50 (DVDD)
- new net +3V3: C10.1, C11.2, C2.1, C3.1, C4.1, C5.1, C6.1, C7.1, C8.1, C9.1, U1.1 (IOVDD), U1.10 (IOVDD), U1.22 (IOVDD), U1.33 (IOVDD), U1.42 (IOVDD), U1.43 (ADC_AVDD), U1.44 (VREG_VIN), U1.48 (USB_VDD), U1.49 (IOVDD), U3.2 (VO)
- new net COL1: SW1.2 (B), SW13.2 (B), SW25.2 (B), SW37.2 (B)
- new net COL10: SW10.2 (B), SW22.2 (B), SW34.2 (B), SW46.2 (B)
- new net COL11: SW11.2 (B), SW23.2 (B), SW35.2 (B), SW47.2 (B)
- new net COL12: SW12.2 (B), SW24.2 (B), SW36.2 (B), SW48.2 (B)
- new net COL2: SW14.2 (B), SW2.2 (B), SW26.2 (B), SW38.2 (B)
- new net COL3: SW15.2 (B), SW27.2 (B), SW3.2 (B), SW39.2 (B)
- new net COL4: SW16.2 (B), SW28.2 (B), SW4.2 (B), SW40.2 (B)
- new net COL5: SW17.2 (B), SW29.2 (B), SW41.2 (B), SW5.2 (B)
- new net COL6: SW18.2 (B), SW30.2 (B), SW42.2 (B), SW6.2 (B)
- new net COL7: SW19.2 (B), SW31.2 (B), SW7.2 (B)
- new net COL8: SW20.2 (B), SW32.2 (B), SW44.2 (B), SW8.2 (B)
- new net COL9: SW21.2 (B), SW33.2 (B), SW45.2 (B), SW9.2 (B)
- new net DATA+: R4.1, U2.6 (I/O2)
- new net DATA-: R3.1, U2.7 (I/O1)
- new net GND: C1.2, C10.2, C11.1, C12.2, C13.2, C14.2, C2.2, C3.2, C4.2, C5.2, C6.2, C7.2, C8.2, C9.2, J1.A1 (GND), J1.A12 (GND), J1.B1 (GND), J1.B12 (GND), R1.2, R2.2, U1.57 (GND), U2.4 (GND), U2.5 (GND), U3.1 (GND)
- new net ROW1: D1.1 (K), D10.1 (K), D11.1 (K), D12.1 (K), D2.1 (K), D3.1 (K), D4.1 (K), D5.1 (K), D6.1 (K), D7.1 (K), D8.1 (K), D9.1 (K)
- new net ROW2: D13.1 (K), D14.1 (K), D15.1 (K), D16.1 (K), D17.1 (K), D18.1 (K), D19.1 (K), D20.1 (K), D21.1 (K), D22.1 (K), D23.1 (K), D24.1 (K)
- new net ROW3: D25.1 (K), D26.1 (K), D27.1 (K), D28.1 (K), D29.1 (K), D30.1 (K), D31.1 (K), D32.1 (K), D33.1 (K), D34.1 (K), D35.1 (K), D36.1 (K)
- new net ROW4: D37.1 (K), D38.1 (K), D39.1 (K), D40.1 (K), D41.1 (K), D42.1 (K), D44.1 (K), D45.1 (K), D46.1 (K), D47.1 (K), D48.1 (K)
- new net VBUS: C1.1, J1.A4 (VBUS), J1.A9 (VBUS), J1.B4 (VBUS), J1.B9 (VBUS), U2.1 (VBUS), U2.8 (VBUS), U3.3 (VI)
- no-connect marks 0 -> 3
Other:
- note added: "Microcontroller -------------"
- note added: "Switch Matrix ----------"
- note added: "USB-C Connection w/ Data Protection ---------------------------"
- note added: "Voltage Regulator -------------"

Commit message: crystals
Parts:
- added X1: ABM8-272-T3, ABM8-272-T3_ABR, symbol 2026-05-21_04-03-18:ABM8-272-T3
Connections:
- net GND: now also X1.4

Commit message: schematic version 1
Parts:
- added C15, C16: 15p, symbol Device:C_Small
- added C17: 100n, symbol Device:C_Small
- added R5, R7: 1k, symbol Device:R_Small
- added R6, R8: 10k, symbol Device:R_Small
- added SW43, SW49: SW_Push, symbol Switch:SW_Push
- added U4: W25Q128JVS, Package_SO:SOIC-8_5.3x5.3mm_P1.27mm, symbol Memory_Flash:W25Q128JVS
Connections:
- net +3V3: now also C17.1, R6.1, R8.1, U4.8 (VCC)
- net COL1: now also U1.6 (GPIO4)
- net COL10: now also U1.16 (GPIO13)
- net COL11: now also U1.17 (GPIO14)
- net COL12: now also U1.18 (GPIO15)
- net COL2: now also U1.7 (GPIO5)
- net COL3: now also U1.8 (GPIO6)
- net COL4: now also U1.9 (GPIO7)
- net COL5: now also U1.11 (GPIO8)
- net COL6: now also U1.12 (GPIO9)
- net COL7: now also U1.13 (GPIO10)
- net COL8: now also U1.14 (GPIO11)
- net COL9: now also U1.15 (GPIO12)
- net GND: now also J1.SH (SHIELD), U1.19 (TESTEN), X1.2, C15.1, C16.2, C17.2, SW43.1, SW49.1, U4.4 (GND)
- net ROW1: now also U1.2 (GPIO0)
- net ROW2: now also U1.3 (GPIO1)
- net ROW3: now also U1.4 (GPIO2)
- net ROW4: now also U1.5 (GPIO3)
- net XIN: now reaches X1.1
- net XIN: now also U1.20 (XIN), C15.2
- net at X1.3: now also C16.1, R5.1
- net XOUT: now reaches U1.21 (XOUT)
- net XOUT: now also R5.2
- net RESET: now reaches U1.26 (RUN)
- net RESET: now also R8.2, SW49.2
- net QSPI_SD3: now reaches U1.51 (QSPI_SD3)
- net QSPI_SD3: now also U4.7 (~{HOLD}/~{RESET}/IO_{3})
- net QSPI_SCLK: now reaches U1.52 (QSPI_SCLK)
- net QSPI_SCLK: now also U4.6 (CLK)
- net QSPI_SD0: now reaches U1.53 (QSPI_SD0)
- net QSPI_SD0: now also U4.5 (DI/IO_{0})
- net QSPI_SD2: now reaches U1.54 (QSPI_SD2)
- net QSPI_SD2: now also U4.3 (~{WP}/IO_{2})
- net QSPI_SD1: now reaches U1.55 (QSPI_SD1)
- net QSPI_SD1: now also U4.2 (DO/IO_{1})
- net QSPI_SS: now reaches U1.56 (~{QSPI_SS})
- net QSPI_SS: now also R6.2, R7.2, U4.1 (~{CS})
- new net BOOT: R7.1, SW43.2
- no-connect marks 3 -> 18
Other:
- note added: "Crystal ------"
- note added: "Flash Memory ----------"
- company: (none) -> 8-bit-studios physics department
- title: (none) -> Pankeyk
- moved on the sheet: C1, C2, U3, X1
