File: pcb/v1/v1.kicad_sch (KiCad schematic)
At the start: 127 parts, among them J1 USB_C_Receptacle_USB2.0_16P, SW1 SW_Push, SW2 SW_Push, U1 NCP1117-3.3_SOT223, U2 USB6B1, U3 W25Q128JVS, U4 RP2040, X1 ABM8-272-T3

Commit message: bottom case rev 1 and pcb updates
Parts:
- removed U1: NCP1117-3.3_SOT223, Package_TO_SOT_SMD:SOT-223-3_TabPin2, symbol Regulator_Linear:NCP1117-3.3_SOT223
- removed U2: USB6B1, Package_SO:SOIC-8_3.9x4.9mm_P1.27mm, symbol Power_Protection:USB6B1
- added S1: choc_stab, PCM_marbastlib-xp-choc:STAB_choc_2u, symbol PCM_marbastlib-choc:choc_stab
- added U1: USBLC6-2SC6, Package_TO_SOT_SMD:SOT-23-6, symbol Power_Protection:USBLC6-2SC6
- added U5: AP2112K-3.3, Package_TO_SOT_SMD:SOT-23-5, symbol Regulator_Linear:AP2112K-3.3
- C1, C10, C11, C12, C13, C14, C15, C16, C17, C4, C5, C6, C7, C8, C9: footprint (none) -> Capacitor_SMD:C_0402_1005Metric
- C2, C3: value 10u -> 1u; footprint (none) -> Capacitor_SMD:C_0402_1005Metric
- U3: footprint Package_SO:SOIC-8_5.3x5.3mm_P1.27mm -> Package_SON:WSON-8-1EP_6x5mm_P1.27mm_EP3.4x4.3mm; symbol Memory_Flash:W25Q128JVS -> Memory_Flash:W25Q128JVP
Connections:
- net +3V3: now also U5.5 (VOUT)
- net DATA+: now also U1.4 (I/O2)
- net DATA-: now also U1.6 (I/O1)
- net GND: now also U3.9 (EP), U1.2 (GND), U5.2 (GND)
- net VBUS: now also U1.5 (VBUS), U5.1 (VIN), U5.3 (EN)
- net at J1.A7 (D-), J1.B7 (D-): now also U1.1 (I/O1)
- net at J1.A6 (D+), J1.B6 (D+): now also U1.3 (I/O2)
- net RPD-: now reaches R8.2, U4.47 (USB_DP)
- net RPD+: now reaches R7.2, U4.46 (USB_DM)
Other:
- moved on the sheet: R7, R8

Commit message: pcb v1
Connections:
- net COL1: now also U4.17 (GPIO14); no longer U4.6 (GPIO4)
- net COL10: now also U4.5 (GPIO3); no longer U4.16 (GPIO13)
- net COL11: now also U4.4 (GPIO2); no longer U4.17 (GPIO14)
- net COL12: now also U4.3 (GPIO1); no longer U4.18 (GPIO15)
- net COL2: now also U4.18 (GPIO15); no longer U4.7 (GPIO5)
- net COL3: now also U4.29 (GPIO18); no longer U4.8 (GPIO6)
- net COL4: now also U4.38 (GPIO26/ADC0); no longer U4.9 (GPIO7)
- net COL5: now also U4.2 (GPIO0); no longer U4.11 (GPIO8)
- net COL6: now also U4.35 (GPIO23); no longer U4.12 (GPIO9)
- net COL7: now also U4.36 (GPIO24); no longer U4.13 (GPIO10)
- net COL8: now also U4.6 (GPIO4); no longer U4.14 (GPIO11)
- net COL9: now also U4.7 (GPIO5); no longer U4.15 (GPIO12)
- net ROW1: now also U4.30 (GPIO19); no longer U4.2 (GPIO0)
- net ROW2: now also U4.31 (GPIO20); no longer U4.3 (GPIO1)
- net ROW3: now also U4.16 (GPIO13); no longer U4.4 (GPIO2)
- net ROW4: now also U4.15 (GPIO12); no longer U4.5 (GPIO3)

Commit message: pcb v1
Parts:
- added H1, H2, H3, H4, H5, H6, H7, H8: M2, MountingHole:MountingHole_2.2mm_M2_Pad, symbol Mechanical:MountingHole_Pad
Connections:
- net GND: now also H1.1, H2.1, H3.1, H4.1, H5.1, H6.1, H7.1, H8.1

Commit message: pcb BOM updates
Parts:
- C1, C11, C12, C14, C15, C16, C17, C6, C7, C8, C9: LCSC (none) -> 0402B104J160CT
- C10, C13, C2, C3: LCSC (none) -> GRM155Z71A105KE01D
- C4, C5: LCSC (none) -> GRM1555C1H150FA01D
- D1, D10, D11, D12, D13, D14, D15, D16, D17, D18, D19, D2, D20, D21, D22, D23, D24, D25, D26, D27, D28, D29, D3, D30, D31, D32, D33, D34, D35, D36, D37, D38, D39, D4, D40, D41, D42, D43, D44, D45, D46, D47, D5, D6, D7, D8, D9: LCSC (none) -> 1N4148WS
- H1, H2, H3, H4, H5, H6, H7, H8: now not fitted
- J1: LCSC (none) -> TYPE-C-31-M-12
- MX1, MX10, MX11, MX12, MX13, MX14, MX15, MX16, MX17, MX18, MX19, MX2, MX20, MX21, MX22, MX23, MX24, MX25, MX26, MX27, MX28, MX29, MX3, MX30, MX31, MX32, MX33, MX34, MX35, MX36, MX37, MX38, MX39, MX4, MX40, MX41, MX42, MX43, MX44, MX45, MX46, MX47, MX5, MX6, MX7, MX8, MX9: LCSC (none) -> CPG151101S11-2
- R1, R2: LCSC (none) -> CRCW04025K10JNED
- R3, R6: LCSC (none) -> CRCW040210K0FKEDC
- R4, R5: LCSC (none) -> CRCW04021K00FKED
- R7, R8: LCSC (none) -> CRCW040227R0FKED
- S1: now not fitted; now left out of the parts list
- SW1, SW2: LCSC (none) -> TL3342F160QG
- U1: LCSC (none) -> USBLC6-2SC6
- U3: value W25Q128JVS -> W25Q128JVP; LCSC (none) -> W25Q128JVP
- U4: LCSC (none) -> RP2040
- U5: LCSC (none) -> AP2112K-3.3
- X1: LCSC (none) -> ABM8-272-T3
Connections:
- net ROW4: now also U4.8 (GPIO6); no longer U4.15 (GPIO12)
