File: pcb/v1/_restore_backup_2026-05-21T23-04-20-848/v1.kicad_sch (KiCad schematic)
At the start: 127 parts, among them J1 USB_C_Receptacle_USB2.0_16P, SW1 SW_Push, SW2 SW_Push, U1 NCP1117-3.3_SOT223, U2 USB6B1, U3 W25Q128JVS, U4 RP2040, X1 ABM8-272-T3

Commit message: pcb
Parts:
- J1: footprint Connector_USB:USB_C_Receptacle_HRO_TYPE-C-31-M-12 -> (none)
- R1, R2, R3, R4, R5, R6, R7, R8: footprint Resistor_SMD:R_0402_1005Metric -> (none)
- SW1, SW2: footprint Button_Switch_SMD:SW_SPST_TL3342 -> (none)
- X1: footprint Crystal:Crystal_SMD_Abracon_ABM8G-4Pin_3.2x2.5mm -> ABM8-272-T3_ABR
- renumbered D1 to D48, D2 to D49, D3 to D50, D4 to D51, D5 to D52, D6 to D53, D7 to D54, D8 to D55, D9 to D56, D10 to D57, D11 to D58, D12 to D59, D13 to D60, D14 to D61, D15 to D62, D16 to D63, D17 to D64, D18 to D65, D19 to D66, D20 to D67, D21 to D68, D22 to D69, D23 to D70, D24 to D71, D25 to D72, D26 to D73, D27 to D74, D28 to D75, D29 to D76, D30 to D77, D31 to D78, D32 to D79, D33 to D80, D34 to D81, D35 to D82, D36 to D83, D37 to D84, D38 to D85, D39 to D86, D40 to D87, D41 to D88, D42 to D89, D43 to D91, D44 to D92, D45 to D93, D46 to D94, D47 to D95, MX43 to MX44, MX44 to MX45, MX45 to MX46, MX46 to MX47, MX47 to MX48
Other:
- moved on the sheet: C4, C5, R5, X1
