File: pcb/gasket-mount/matrix/matrix.kicad_pcb (KiCad board)
At the start: 2 copper layers, 228.6 x 76.2 mm, 104 parts

Commit message: fixed switches with extra 3D models
Parts:
- MX1, MX10, MX11, MX12, MX13, MX14, MX15, MX16, MX17, MX18, MX19, MX2, MX20, MX21, MX22, MX23, MX24, MX25, MX26, MX27, MX28, MX29, MX3, MX30, MX31, MX32, MX33, MX34, MX35, MX36, MX37, MX38, MX39, MX4, MX40, MX41, MX42, MX43, MX44, MX45, MX46, MX47, MX5, MX6, MX7, MX8, MX9: footprint PCM_marbastlib-mx:SW_MX_HS_CPG151101S11_1u -> Switch_lib:SW_MX_HS_CPG151101S11_1u
- S1: footprint PCM_marbastlib-xp-choc:STAB_choc_2u -> Switch_lib:STAB_choc_2u
Routing:
- net Net-(D42-A): track 0.54 -> 4.62 mm

Commit message: PCB finishing touches
Parts:
- renumbered D19 to D18, D20 to D19, D21 to D20, D22 to D21, D23 to D22, D24 to D23, D18 to D24, D30 to D25, D25 to D26, D26 to D27, D27 to D28, D28 to D29, D29 to D30
Routing:
- net COL7: track 52.5 -> 51.6 mm
- net Net-(D4-A): track 3.43 -> 2.85 mm
- net Net-(D5-A): track 3.43 -> 2.85 mm
- net Net-(D6-A): track 3.43 -> 2.85 mm
- net Net-(D7-A): track 3.43 -> 2.85 mm
- net Net-(D8-A): track 3.43 -> 2.85 mm
- net Net-(D9-A): track 3.43 -> 2.85 mm
- net Net-(D10-A): track 3.43 -> 2.85 mm
- net Net-(D11-A): track 3.43 -> 2.85 mm
- net Net-(D12-A): track 3.43 -> 2.85 mm
- net Net-(D47-A): track 4.62 -> 4.09 mm
- net Net-(D36-A): track 3.12 -> 2.58 mm
- net Net-(D46-A): track 4.62 -> 4.09 mm
- net Net-(D35-A): track 3.12 -> 2.58 mm
- net Net-(D45-A): track 4.62 -> 4.09 mm
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