File: pcb/gasket-mount/matrix/matrix.kicad_sch (KiCad schematic)
At the start: 104 parts

Commit message: PCB finishing touches
Parts:
- MX1, MX10, MX11, MX12, MX13, MX14, MX15, MX16, MX17, MX18, MX19, MX2, MX20, MX21, MX22, MX23, MX24, MX25, MX26, MX27, MX28, MX29, MX3, MX30, MX31, MX32, MX33, MX34, MX35, MX36, MX37, MX38, MX39, MX4, MX40, MX41, MX42, MX43, MX44, MX45, MX46, MX47, MX5, MX6, MX7, MX8, MX9: footprint PCM_marbastlib-mx:SW_MX_HS_CPG151101S11_1u -> Switch_lib:SW_MX_HS_CPG151101S11_1u
- S1: footprint PCM_marbastlib-xp-choc:STAB_choc_2u -> Switch_lib:STAB_choc_2u
- renumbered D19 to D18, D20 to D19, D21 to D20, D22 to D21, D23 to D22, D24 to D23, D18 to D24, D30 to D25, D25 to D26, D26 to D27, D27 to D28, D28 to D29, D29 to D30
Other:
- note added: "CONNECTOR"
- note added: "MOUNTING"
- note added: "SWITCH MATRIX"
- note removed: "Connector -------"
- note removed: "Mounting -------"
- note removed: "Switch Matrix ----------"
- moved on the sheet: D1, D10, D11, D12, D13, D14, D15, D16, D17, D18, D19, D2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

Commit message: I finally ordered\!
Parts:
- U1: value (none) -> TF31-18S-0.5SH(800)
Changed lines of the file:
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@@
 			)
 		)
-		(property "Value" ""
+		(property "Value" "TF31-18S-0.5SH(800)"
 			(at 248.92 91.44 0)
 			(show_name no)
