File: pcb/gasket-mount/controller/controller.kicad_sch (KiCad schematic)
At the start: 137 parts, among them J1 USB_C_Receptacle_USB2.0_16P, J2 Conn_01x18_MountingPin, SW1 SW_Push, SW2 SW_Push, U1 USBLC6-2SC6, U3 W25Q128JVP, U4 RP2040, U5 AP2112K-3.3, X1 ABM8-272-T3

Commit message: Netclasses and ready for updated pcb layout
Parts:
- removed J2: Conn_01x18_MountingPin, Connector_Samtec_MicroMate:Samtec_T1M-18-X-S-V_1x18-1MP_P1.0mm_Terminal_Vertical, symbol Connector_Generic_MountingPin:Conn_01x18_MountingPin
- added U2: (no value), EasyEDA_Lib:FPC-SMD_18P-P0.50_TF31-18S-0.5SH-800, symbol EasyEDA_Lib:TF31-18S-0.5SH(800)_C3168422
Connections:
- net COL1: now also U4.11 (GPIO8); no longer U4.17 (GPIO14)
- net COL2: now also U4.12 (GPIO9); no longer U4.18 (GPIO15)
- net COL3: now also U4.13 (GPIO10); no longer U4.29 (GPIO18)
- net ROW1: now also U4.14 (GPIO11); no longer U4.30 (GPIO19)
- net ROW3: now also U4.9 (GPIO7); no longer U4.16 (GPIO13)
- net RPD+: now also R8.2, U4.47 (USB_DP); no longer R7.2, U4.46 (USB_DM)
- net RPD-: now also R7.2, U4.46 (USB_DM); no longer R8.2, U4.47 (USB_DP)
- net USB-: now reaches J1.A7 (D-), J1.B7 (D-), U1.1 (I/O1)
- net USB+: now reaches J1.A6 (D+), J1.B6 (D+), U1.3 (I/O2)

Commit message: Compact form factor
Parts:
- removed D1, D10, D11, D12, D13, D14, D15, D16, D17, D18, D19, D2, D20, D21, D22, D23, D24, D25, D26, D27, D28, D29, D3, D30, D31, D32, D33, D34, D35, D36, D37, D38, D39, D4, D40, D41, D42, D43, D44, D45, D46, D47, D5, D6, D7, D8, D9: 1N4148WS, Diode_SMD:D_SOD-323, symbol Diode:1N4148WS
- removed H1, H2, H3, H4, H5, H6, H7, H8: M2, MountingHole:MountingHole_2.2mm_M2_Pad, symbol Mechanical:MountingHole_Pad
- removed MX1, MX10, MX11, MX12, MX13, MX14, MX15, MX16, MX17, MX18, MX19, MX2, MX20, MX21, MX22, MX23, MX24, MX25, MX26, MX27, MX28, MX29, MX3, MX30, MX31, MX32, MX33, MX34, MX35, MX36, MX37, MX38, MX39, MX4, MX40, MX41, MX42, MX43, MX44, MX45, MX46, MX47, MX5, MX6, MX7, MX8, MX9: MX_SW_HS, PCM_marbastlib-mx:SW_MX_HS_CPG151101S11_1u, symbol PCM_marbastlib-mx:MX_SW_HS_CPG151101S11
- removed S1: choc_stab, PCM_marbastlib-xp-choc:STAB_choc_2u, symbol PCM_marbastlib-choc:choc_stab
- removed SW1, SW2: SW_Push, Button_Switch_SMD:SW_SPST_TL3342, symbol Switch:SW_Push
- added SW2, SW3: (no value), EasyEDA_Lib:KEY-SMD_4P-L4.2-W3.2-P2.20-LS4.6, symbol EasyEDA_Lib:SKRPAME010
Connections:
- net BOOT: now also SW2.1, SW2.2
- net COL1: now also U2.10
- net COL10: now also U2.5
- net COL11: now also U2.4
- net COL12: now also U2.3
- net COL2: now also U2.11
- net COL3: now also U2.12
- net COL4: now also U2.17, U4.18 (GPIO15); no longer U4.38 (GPIO26/ADC0)
- net COL5: now also U2.2
- net COL6: now also U2.15, U4.16 (GPIO13); no longer U4.35 (GPIO23)
- net COL7: now also U2.16, U4.17 (GPIO14); no longer U4.36 (GPIO24)
- net COL8: now also U2.6
- net COL9: now also U2.7
- net GND: now also U2.1, U2.18, U2.19, U2.20, SW2.3, SW2.4, SW3.3, SW3.4
- net RESET: now also SW3.1, SW3.2
- net ROW1: now also U2.13
- net ROW2: now also U2.14, U4.15 (GPIO12); no longer U4.31 (GPIO20)
- net ROW3: now also U2.9
- net ROW4: now also U2.8
Other:
- moved on the sheet: U2

Commit message: Last commit before changing Flash memory
Parts:
- added H1, H2, H3: MountingHole_Pad, MountingHole:MountingHole_2.2mm_M2_ISO14580_Pad, symbol Mechanical:MountingHole_Pad
Connections:
- net GND: now also H1.1, H2.1, H3.1

Commit message: new flash
Parts:
- removed C1: 100n, Capacitor_SMD:C_0402_1005Metric, symbol Device:C_Small
- removed H2: MountingHole_Pad, MountingHole:MountingHole_2.2mm_M2_ISO14580_Pad, symbol Mechanical:MountingHole_Pad
- removed R3: 10k, Resistor_SMD:R_0402_1005Metric, symbol Device:R_Small
- removed R4: 1k, Resistor_SMD:R_0402_1005Metric, symbol Device:R_Small
- removed SW2: (no value), EasyEDA_Lib:KEY-SMD_4P-L4.2-W3.2-P2.20-LS4.6, symbol EasyEDA_Lib:SKRPAME010
- removed U3: W25Q128JVP, Package_SON:WSON-8-1EP_6x5mm_P1.27mm_EP3.4x4.3mm, symbol Memory_Flash:W25Q128JVP
- added C18: 100n, Capacitor_SMD:C_0402_1005Metric, symbol Device:C_Small
- added R10: 10k, Resistor_SMD:R_0402_1005Metric, symbol Device:R_Small
- added R9: 1k, Resistor_SMD:R_0402_1005Metric, symbol Device:R_Small
- added SW4: (no value), EasyEDA_Lib:KEY-SMD_4P-L4.2-W3.2-P2.20-LS4.6, symbol EasyEDA_Lib:SKRPAME010
- added U6: (no value), EasyEDA_Lib:USON-8_L3.0-W2.0-P0.50-BL-EP, symbol EasyEDA_Lib:W25Q16JVUXIQ
Connections:
- net +3V3: now also C18.1, R10.2, U6.8 (VCC)
- net BOOT: now also R9.1, SW4.1, SW4.2
- net GND: now also C18.2, SW4.3, SW4.4, U6.4 (GND), U6.9 (EP)
- net QSPI_SCLK: now also U6.6 (CLK)
- net QSPI_SD0: now also U6.5 (DI(IO0))
- net QSPI_SD1: now also U6.2 (DO(IO1))
- net QSPI_SD2: now also U6.3 (WP#(IO2))
- net QSPI_SD3: now also U6.7 (HOLD#orRESET#(IO3))
- net QSPI_SS: now also R10.1, R9.2, U6.1 (CS#)
Other:
- moved on the sheet: H1, H3

Commit message: PCB finishing touches
Parts:
- removed SW3: (no value), EasyEDA_Lib:KEY-SMD_4P-L4.2-W3.2-P2.20-LS4.6, symbol EasyEDA_Lib:SKRPAME010
- added H3: Mount, MountingHole:MountingHole_2.2mm_M2_ISO14580_Pad, symbol Mechanical:MountingHole_Pad
- added J2: I2C, Connector_PinHeader_2.54mm:PinHeader_1x02_P2.54mm_Vertical, symbol Connector:Conn_01x02_Pin
- added J3: PWR, Connector_PinHeader_2.54mm:PinHeader_1x02_P2.54mm_Vertical, symbol Connector:Conn_01x02_Pin
- added SW1: (no value), EasyEDA_Lib:KEY-SMD_4P-L4.2-W3.2-P2.20-LS4.6, symbol EasyEDA_Lib:SKRPAME010
- H1: value MountingHole_Pad -> Mount
- H2: renamed from H3; value MountingHole_Pad -> Mount
- J1: value USB_C_Receptacle_USB2.0_16P -> TYPE-C-31-M-12
- U2: value (none) -> TF31-18S-0.5SH(800)
- renumbered SW4 to SW2
Connections:
- net +3V3: now also J3.2 (Pin_2)
- net COL1: now also U2.6, U4.6 (GPIO4); no longer U2.10, U4.11 (GPIO8)
- net COL10: now also U2.15, U4.16 (GPIO13); no longer U2.5, U4.5 (GPIO3)
- net COL11: now also U2.16, U4.17 (GPIO14); no longer U2.4, U4.4 (GPIO2)
- net COL12: now also U2.17, U4.18 (GPIO15); no longer U2.3, U4.3 (GPIO1)
- net COL2: now also U2.7, U4.7 (GPIO5); no longer U2.11, U4.12 (GPIO9)
- net COL3: now also U2.8, U4.8 (GPIO6); no longer U2.12, U4.13 (GPIO10)
- net COL4: now also U2.9, U4.9 (GPIO7); no longer U2.17, U4.18 (GPIO15)
- net COL5: now also U2.10, U4.11 (GPIO8); no longer U2.2, U4.2 (GPIO0)
- net COL6: now also U2.11, U4.12 (GPIO9); no longer U2.15, U4.16 (GPIO13)
- net COL7: now also U2.12, U4.13 (GPIO10); no longer U2.16, U4.17 (GPIO14)
- net COL8: now also U2.13, U4.14 (GPIO11); no longer U2.6, U4.6 (GPIO4)
- net COL9: now also U2.14, U4.15 (GPIO12); no longer U2.7, U4.7 (GPIO5)
- net GND: now also H3.1, J3.1 (Pin_1), SW1.3, SW1.4
- net RESET: now also SW1.1, SW1.2
- net ROW1: now also U2.5, U4.5 (GPIO3); no longer U2.13, U4.14 (GPIO11)
- net ROW2: now also U2.4, U4.4 (GPIO2); no longer U2.14, U4.15 (GPIO12)
- net ROW3: now also U2.3, U4.3 (GPIO1); no longer U2.9, U4.9 (GPIO7)
- net ROW4: now also U2.2, U4.2 (GPIO0); no longer U2.8, U4.8 (GPIO6)
- net GPIO26/SDA: now reaches U4.38 (GPIO26/ADC0)
- net GPIO26/SDA: now also J2.1 (Pin_1)
- net GPIO27/SCL: now reaches U4.39 (GPIO27/ADC1)
- net GPIO27/SCL: now also J2.2 (Pin_2)
- no-connect marks 18 -> 16
Other:
- note added: "16Mb QSPI"
- note added: "5V to 3.3V"
- note added: "<- Place this close to pin 44"
- note added: "CONNECTOR"
- note added: "CRYSTAL"
- note added: "Decoupling capacitors"
- note added: "Expose power and an I2C bus for debigging"
- note added: "FLASH MEMORY"
- note added: "M2 Screws"
- note added: "MICROCONTROLLER"
- note added: "MOUNTING"
- note added: "Place each close to an RP2040 power pin"
- note added: "RP2040"
- note added: "Test Points"
- note added: "To switch matrix"
- note added: "USB-C CONNECTOR"
- note added: "VOLTAGE REGULATOR"
- note added: "With data protection"
- note removed: "Crystal ------"
- note removed: "Flash Memory ----------"
- note removed: "Microcontroller -------------"
- note removed: "Switch Matrix ----------"
- note removed: "USB-C Connection w/ Data Protection ---------------------------"
- note removed: "Voltage Regulator -------------"
- moved on the sheet: C10, C11, C12, C13, C14, C15, C16, C17, C18, C2, C3, C4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

Commit message: I finally ordered\!
Parts:
- C10, C13: LCSC GRM155Z71A105KE01D -> C52923
- C11, C12, C14, C15, C16, C17, C18, C6, C7, C8, C9: LCSC 0402B104J160CT -> C1525
- C2, C3: value 1u -> 10u; footprint Capacitor_SMD:C_0402_1005Metric -> Capacitor_SMD:C_0603_1608Metric; LCSC GRM155Z71A105KE01D -> C96446
- C4, C5: LCSC GRM1555C1H150FA01D -> C1548
- R1, R2: value 5k1 -> 5.1k; LCSC CRCW04025K10JNED -> C25905
- R10, R6: LCSC CRCW040210K0FKEDC -> C25744
- R5, R9: LCSC CRCW04021K00FKED -> C11702
- R7, R8: value 27.4 -> 33; LCSC CRCW040227R0FKED -> C25105
- SW1, SW2: value (none) -> SKRPAME010; LCSC (none) -> C19724063; LCSC Part Name 轻触开关 -> (none)
- U6: value (none) -> W25Q16JVUXIQ; LCSC (none) -> C2843335; LCSC Part Name 支持双/四路SPI接口的3V、16Mbit 串行闪存 -> (none)
